File: Eagle/MICHA.brd (EAGLE design)
At the start: 110.5 x 83.1 mm, 57 parts, among them IC1 LM4041A12LP, K1 PIN20X2, T1 BSS84, U1 ARDUINO_MKR_ZERO, U2 MIKROE_CLICK, X1 RJ45-RJULE4318101, X2 RJ45-RJULE4318101, X3 RJ45-RJULE4318101, X4 RJ45-RJULE4318101, X5 RJ45-RJULE4318101, X6 RJ45-RJULE4318101, X7 BUCHANAN_4_3.5MM

Commit message: MICHAv2.0
Version 2.0 de MICHA
Parts:
- removed D1: STMICROELECTRONICS_STPS1L30ASTMICROELECTRONICS_STPS1L30A_0_0, Diode_STPS1L30A:STMICROELECTRONICS_STPS1L30A_0
- removed TVS3: 5Vdc/12pF, EMCComponents (rev19b):WE-TVS_SOT23-3L
- removed Z4, Z5: 3,3V, Zener_SMA:ZENER_SMA
- added DS1, DS2, DS3, DS4: SDM10M45SD, SchottkyDiodes_SDM10M45SD:SDM10M45SD_SOT-26
- added JP1, JP2: (no value), jumper:JP2Q
- added O1: HMHA281R2, HMHA281R2:HMHA281R2
- added R18: 390, resistor:R1206
- added R19: 2k, resistor:R1206
- added R20, R21, R22, R23, R24, R25: 33, resistor:R1206
- added U3: MAX4528CSA, MAX4528CSA:SOIC127P600X175-8N
- added X8: MPT_0,5/_2-2,54_1725656_2, MPT_0_5__2-2_54_1725656:PH_MPT_0,5/_2-2,54_1725656
- R1, R2: value 180 -> 100
- R12, R8, R9: device rcl:R1210 -> rcl:R1206
- R6: value 2k -> 680
- R7: value 2k -> 1k
- TVS1, TVS2: value 5Vdc/12pF -> TVS_SOD123; device EMCComponents (rev19b):WE-TVS_SOT23-3L -> TV02W6V0B-G_SOD123:TVS_SOD123
- U2: value MIKROE_CLICK -> MIKROE_CLICK_UPGRADE; device mikrobus_lib:MIKROE_BUS_MIDI_NOLABEL -> mikrobus_lib:MIKROE_BUS_MIDI_UPGRADE
- X1, X2, X3, X4, X5, X6: value RJ45-RJULE4318101 -> SS-7188S-A-NF_V2; device con-amphenol-rj45-ld:RJ45-RJULE4318101 -> SS-7188S-A-NF:BEL_SS-7188S-A-NF
- Z1, Z2: value 5,1V/1W -> 5,1V-1W
- moved R7 54.9 mm to (49.5, 5.08), turned to 0 degrees
- moved Z3 43.5 mm to (22.4, 44.5), turned to 90 degrees
- moved R6 39.1 mm to (61.9, -4.13), turned to 180 degrees
- moved C1 19.0 mm to (22.9, 20.3), turned to 180 degrees
- moved R11 18.1 mm to (49.5, -3.81)
- moved C12 17.0 mm to (49.5, -0.79), turned to 180 degrees
- moved IC1 16.5 mm to (16.7, 17.5), turned to 90 degrees
- moved T1 16.4 mm to (29.8, 21.7), turned to 0 degrees
- moved TVS1 15.9 mm to (10.5, -2.22), turned to 0 degrees
- moved C13 14.9 mm to (61.9, -1.27)
- moved C15 14.8 mm to (19.4, 29.5), turned to 270 degrees
- moved C9 14.6 mm to (61.9, 13.7)
- moved R12 14.5 mm to (22.9, 17.5), turned to 0 degrees
- moved C10 14.3 mm to (61.9, 10.8)
- moved C11 14.0 mm to (61.9, 7.94)
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Connections:
- net SOL_WARM renamed SOL_HOT
- net VALVE1_CLOSE renamed VALVE1_DIR
- net VALVE1_OPEN renamed VALVE1_POWER
- net VALVE2_CLOSE renamed VALVE2_DIR
- net VALVE2_OPEN renamed VALVE2_POWER
- removed net +3V3: C15.1, D1.1, K1.1, U2.P$7
- removed net AN: AN.1, U2.P$1
- removed net MISO: R10.2, U2.P$5
- removed net PUMP_SERVO: R6.1, X4.6
- new net N$10: U2.A, U3.1
- new net N$11: C11.1, DS1.3, R13.2, R20.1, U1.J4_5
- new net N$12: C10.1, DS1.6, R14.2, R21.1, U1.J4_6
- new net N$13: C9.1, DS2.3, R15.2, R22.1, U1.J4_7
- new net N$15: R10.2, U2.R_MISO
- new net N$16: AN.1, U2.R_AN
- new net N$17: R24.2, X8.2
- new net N$18: R25.2, X8.1
- new net N$19: JP1.4, X5.6
- new net N$20: JP1.2, X3.2
- new net N$21: JP2.4, X5.8
- new net N$22: JP2.2, X3.4
- new net N$7: O1.P$1, R18.2
- new net N$9: C13.1, O1.P$4, R6.1, U1.J4_4
- new net PUMP_SERVO_A+: R18.1, X4.6
- new net PUMP_SERVO_A-: O1.P$2, X4.3
- new net R_SWITCH: K1.36, U3.4
- new net R_X: R24.1, TVS1.P$1, U3.7
- new net R_Y: R25.1, TVS2.P$1, U3.6
- new net VDD: DS1.2, DS1.5, DS2.2, DS2.5, DS3.2, DS3.5, DS4.2, DS4.5, R17.2, R6.2, T1.2, U1.J5_12
- net +5V: now also C15.1, K1.4, U2.R_5V, U3.8; no longer U2.P$10
- net CS: now also U2.R_CS; no longer U2.P$3
- net D0: now also TBD2.4; no longer TBD2.6
- net D19: now also R19.2, U1.J4_3; no longer TVS3.1, U1.J4_6, Z4.C
- net D2: now also TBD2.6; no longer TBD2.4
- net D21: now also U1.J4_2; no longer U1.J4_8
- net GND: now also DS1.1, DS1.4, DS2.1, DS2.4, DS3.1, DS3.4, DS4.1, DS4.4, O1.P$3, R19.1, TVS1.P$2, TVS2.P$2, U2.R_GND1, U2.R_GND2, U3.3, U3.5, X1.S1, X1.S2, X2.S1, X2.S2, X3.S1, X3.S2, X4.S1, X4.S2, X5.S1, X5.S2, X6.S1, X6.S2; no longer TVS1.3, TVS2.3, TVS3.3, U2.P$8, U2.P$9, X1.GND1, X1.GND2, X2.GND1, X2.GND2, X3.GND1, X3.GND2, X4.3, X4.GND1, X4.GND2, X5.GND1, X5.GND2, X6.GND1, X6.GND2, Z4.A, Z5.A
- net N$1: now also U2.B, U3.2; no longer R17.2, T1.2, U1.J5_12
- net N$14: now also C8.1, DS2.6, R16.2, R23.1, U1.J4_8; no longer C13.1, R6.2, TVS3.2, U1.J4_7, Z3.C
- net PI_STOP_BTN: now also DS4.3
- net PUMP_PAUSE_BTN: now also DS3.6
- net PUMP_RELAY: now also JP1.1, JP1.3; no longer X5.6
- net PUMP_START_BTN: now also DS3.3
- net RESERVE: now also JP2.1, JP2.3; no longer X5.8
- net S1/PWM: now also U2.R_PWM; no longer U2.P$16
- net S2/INT: now also U2.R_INT; no longer U2.P$15
- net S3/RST: now also U2.R_RST; no longer U2.P$2
- net SCK: now also U2.R_SCK; no longer U2.P$4
- net SDO: now also Z3.C; no longer D1.2, Z5.C
- net THERMI1: now also R20.2; no longer C11.1, R13.2, TVS2.1, U1.J4_2
- net THERMI2: now also R21.2; no longer C10.1, R14.2, TVS2.2, U1.J4_3
- net THERMI3: now also R22.2; no longer C9.1, R15.2, TVS1.1, U1.J4_4
- net THERMI4: now also R23.2; no longer C8.1, R16.2, TVS1.2, U1.J4_5
Routing:
- net VDD: track 0.00 -> 170.5 mm, vias 0 -> 8
- net D19: track 87.2 -> 10.7 mm
- net N$11: track 0.00 -> 75.9 mm
- net N$12: track 0.00 -> 74.6 mm
- net N$13: track 0.00 -> 69.6 mm
- net N$9: track 0.00 -> 66.2 mm, vias 0 -> 2
- net PUMP_ERR: track 4.47 -> 66.4 mm, vias 0 -> 1
- net R_SWITCH: track 0.00 -> 61.8 mm, vias 0 -> 1
- net THERMI2: track 65.6 -> 5.51 mm
- net THERMI1: track 66.2 -> 8.39 mm
- net THERMI3: track 61.6 -> 5.25 mm
- net THERMI4: track 58.5 -> 6.82 mm
- net R_X: track 0.00 -> 40.1 mm, vias 0 -> 2
- net R_Y: track 0.00 -> 32.9 mm
- net N$19: track 0.00 -> 32.8 mm
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Other:
- board text added: "+12V"
- board text added: "+5V"
- board text added: "GND"
- board text added: "MICHA V2.0"
- board text added: "github.com/AKUINO/MICHA"
- board text removed: "MICHA V1.0"
