File: Eagle/MICHA.sch (EAGLE design)
At the start: 57 parts, among them IC1 LM4041A12LP, K1 PIN20X2, T1 BSS84, U1 ARDUINO_MKR_ZERO, U2 MIKROE_CLICK, X1 RJ45-RJULE4318101, X2 RJ45-RJULE4318101, X3 RJ45-RJULE4318101, X4 RJ45-RJULE4318101, X5 RJ45-RJULE4318101, X6 RJ45-RJULE4318101, X7 BUCHANAN_4_3.5MM

Commit message: MICHAv2.0
Version 2.0 de MICHA
Parts:
- removed D1: STMICROELECTRONICS_STPS1L30ASTMICROELECTRONICS_STPS1L30A_0_0, Diode_STPS1L30A:STMICROELECTRONICS_STPS1L30ASTMICROELECTRONICS_STPS1L30A_0_0
- removed TVS3: 5Vdc/12pF, EMCComponents (rev19b):WE-TVS_SOT23-3L_824022
- removed Z4, Z5: 3,3V, Zener_SMA:ZENER_SMA
- added DS1, DS2, DS3, DS4: SDM10M45SD, SchottkyDiodes_SDM10M45SD:SDM10M45SD
- added JP1, JP2: (no value), jumper:JP2QE
- added O1: HMHA281R2, HMHA281R2:HMHA281R2
- added R18: 390, resistor:R-EU_R1206
- added R19: 2k, resistor:R-EU_R1206
- added R20, R21, R22, R23, R24, R25: 33, resistor:R-EU_R1206
- added U3: MAX4528CSA, MAX4528CSA:MAX4528CSA
- added X8: MPT_0,5/_2-2,54_1725656_2, MPT_0_5__2-2_54_1725656:MPT_0,5/_2-2,54_1725656_2
- R1, R2: value 180 -> 100
- R12, R8, R9: device rcl:R-EU_R1210 -> rcl:R-EU_R1206
- R6: value 2k -> 680
- R7: value 2k -> 1k
- TVS1, TVS2: value 5Vdc/12pF -> TVS_SOD123; device EMCComponents (rev19b):WE-TVS_SOT23-3L_824022 -> TV02W6V0B-G_SOD123:TVS_SOD123
- U2: value MIKROE_CLICK -> MIKROE_CLICK_UPGRADE; device mikrobus_lib:MIKROE_CLICK -> mikrobus_lib:MIKROE_CLICK_UPGRADE
- X1, X2, X3, X4, X5, X6: value RJ45-RJULE4318101 -> SS-7188S-A-NF_V2; device con-amphenol-rj45-ld:RJ45-RJULE4318101 -> SS-7188S-A-NF:SS-7188S-A-NF_V2
- Z1, Z2: value 5,1V/1W -> 5,1V-1W
Connections:
- net AN renamed N$16
- net MISO renamed N$15
- net SOL_WARM renamed SOL_HOT
- net VALVE1_CLOSE renamed VALVE1_DIR
- net VALVE1_OPEN renamed VALVE1_POWER
- net VALVE2_CLOSE renamed VALVE2_DIR
- net VALVE2_OPEN renamed VALVE2_POWER
- removed net +3V3: C15.1, D1.CATHODE, K1.1, U2.3V3
- removed net PUMP_SERVO: R6.1, X4.6
- new net N$10: U2.A, U3.A
- new net N$11: C11.1, DS1.C1, R13.2, R20.1, U1.A3
- new net N$12: C10.1, DS1.C, R14.2, R21.1, U1.A4
- new net N$13: C9.1, DS2.C1, R15.2, R22.1, U1.A5
- new net N$17: R24.2, X8.KL1
- new net N$18: R25.2, X8.KL
- new net N$19: JP1-2.2, X5.6
- new net N$20: JP1-1.2, X3.2
- new net N$21: JP2-2.2, X5.8
- new net N$22: JP2-1.2, X3.4
- new net N$7: O1.A, R18.2
- new net N$9: C13.1, O1.COL, R6.1, U1.A2
- new net PUMP_SERVO_A+: R18.1, X4.6
- new net PUMP_SERVO_A-: O1.C, X4.3
- new net R_SWITCH: K1.36, U3.IN
- new net R_X: R24.1, TVS1.C, U3.X
- new net R_Y: R25.1, TVS2.C, U3.Y
- new net VDD: DS1.A1, DS1.A4, DS2.A1, DS2.A4, DS3.A1, DS3.A4, DS4.A1, DS4.A4, R17.2, R6.2, T1.S, U1.3V3
- net +5V: now also C15.1, K1.4, U3.V+
- net D0: now also TBD2.4; no longer TBD2.6
- net D19: now also R19.2, U1.A1; no longer TVS3.I/O1, U1.A4, Z4.C
- net D2: now also TBD2.6; no longer TBD2.4
- net D21: now also U1.DAC0/A0; no longer U1.A6
- net GND: now also DS1.A2, DS1.A3, DS2.A2, DS2.A3, DS3.A2, DS3.A3, DS4.A2, DS4.A3, O1.EMIT, R19.1, TVS1.C1, TVS2.C1, U3.GND, U3.V-; no longer TVS1.GND, TVS2.GND, TVS3.GND, X4.3, Z4.A, Z5.A
- net N$1: now also U2.B, U3.B; no longer R17.2, T1.S, U1.3V3
- net N$14: now also C8.1, DS2.C, R16.2, R23.1, U1.A6; no longer C13.1, R6.2, TVS3.I/O2, U1.A5, Z3.C
- net PI_STOP_BTN: now also DS4.C1
- net PUMP_PAUSE_BTN: now also DS3.C
- net PUMP_RELAY: now also JP1-1.1, JP1-2.1; no longer X5.6
- net PUMP_START_BTN: now also DS3.C1
- net RESERVE: now also JP2-1.1, JP2-2.1; no longer X5.8
- net SDO: now also Z3.C; no longer D1.ANODE, Z5.C
- net THERMI1: now also R20.2; no longer C11.1, R13.2, TVS2.I/O1, U1.DAC0/A0
- net THERMI2: now also R21.2; no longer C10.1, R14.2, TVS2.I/O2, U1.A1
- net THERMI3: now also R22.2; no longer C9.1, R15.2, TVS1.I/O1, U1.A2
- net THERMI4: now also R23.2; no longer C8.1, R16.2, TVS1.I/O2, U1.A3
Other:
- note added: "v4.2"
- note removed: "v4.0"
- moved on the sheet: AN, C1, C10, C11, C12, C13, C14, C15, C2, C3, C4, C5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
